Commit message: Update nav2.launch.py for SLAM-mode and remove obsolete map files

File: robotics/robot_description/urdf/amr_real.urdf.xacro (robot description, xacro)
@@ -18,5 +18,5 @@
   <xacro:property name="base_to_axle_z"   value="0.3505"/>  <!-- CAD: base_link height above wheel axle -->
   <!-- LiDAR + IMU mount points on base_link (EDIT to real positions) -->
-  <xacro:property name="lidar_xyz" value="0.35 0 -0.075"/>   <!-- top-centre of chassis; adjust -->
+  <xacro:property name="lidar_xyz" value="0.35 0 0.05"/>   <!-- top-centre of chassis; adjust -->
   <xacro:property name="imu_xyz"   value="0 0 0.0"/>    <!-- near chassis centre; adjust -->
   <!-- ===================================================================

Commit message: configured navigation parameters for localization and mapping in the nav2_params.yaml file, added a new launch file for localization, and included the warehouse map files for navigation. Updated the robot description URDF to reflect changes in the robot model.

File: robotics/robot_description/urdf/amr_real.urdf.xacro (robot description, xacro)
@@ -14,7 +14,7 @@
        >>> VERIFY THESE THREE NUMBERS against your real robot / RViz <<<
        =================================================================== -->
-  <xacro:property name="wheel_radius"     value="0.060"/>   <!-- metres: your drive-wheel radius -->
+  <xacro:property name="wheel_radius"     value="0.080"/>   <!-- metres: measured from DR_Link/DL_Link.STL bounding box (was 0.060, wrong scale -> odom drift) -->
   <xacro:property name="wheel_separation" value="0.5787"/>  <!-- from DL/DR joint origins (2 x 0.28935) -->
-  <xacro:property name="base_to_axle_z"   value="0.3505"/>  <!-- CAD: base_link height above wheel axle -->
+  <xacro:property name="base_to_axle_z"   value="0.3305"/>  <!-- CAD: base_link height above wheel axle (DR/DL joint z = -0.3305) -->
   <!-- LiDAR + IMU mount points on base_link (EDIT to real positions) -->
   <xacro:property name="lidar_xyz" value="0.35 0 0.05"/>   <!-- top-centre of chassis; adjust -->
@@ -68,6 +68,6 @@
       <child_frame_id>base_footprint</child_frame_id>
       <odom_publish_frequency>50</odom_publish_frequency>
-      <max_linear_velocity>1.2</max_linear_velocity>
-      <min_linear_velocity>-1.2</min_linear_velocity>
+      <max_linear_velocity>1.5</max_linear_velocity>
+      <min_linear_velocity>-1.5</min_linear_velocity>
       <max_angular_velocity>1.5</max_angular_velocity>
       <min_angular_velocity>-1.5</min_angular_velocity>
