Commit message: Refine AMR-X materials and LiDAR alignment

File: robotics/robot_description/urdf/AMR-X_robot.urdf (robot description, URDF)
Before this commit: robot AMR-X_robot, 11 links, 10 joints
Links:
- link base_link: geometry collision mesh filename=package://robot_description/meshes/base_link.STL; visual mesh filename=package://robot_description/meshes/base_body_visual.STL

File: robotics/robot_description/urdf/amr_real.urdf.xacro (robot description, xacro)
@@ -18,5 +18,7 @@
   <xacro:property name="base_to_axle_z"   value="0.3305"/>  <!-- CAD: base_link height above wheel axle (DR/DL joint z = -0.3305) -->
   <!-- LiDAR + IMU mount points on base_link (EDIT to real positions) -->
-  <xacro:property name="lidar_xyz" value="0.35 0 0.05"/>   <!-- top-centre of chassis; adjust -->
+  <!-- Front CAD LiDAR puck centre is x=0.3447, y=-0.0044.  Place the
+       simulated scan plane near the puck's optical top surface. -->
+  <xacro:property name="lidar_xyz" value="0.3447 -0.0044 -0.068"/>
   <xacro:property name="imu_xyz"   value="0 0 0.0"/>    <!-- near chassis centre; adjust -->
   <!-- ===================================================================

Commit message: Stabilize robot contact and caster physics

File: robotics/robot_description/urdf/AMR-X_robot.urdf (robot description, URDF)
Before this commit: robot AMR-X_robot, 11 links, 10 joints
Links:
- link BL_Caster_Wheel_Link: geometry collision cylinder length=0.044 radius=0.05; visual mesh filename=package://robot_description/meshes/BL_Caster_Wheel_Link.STL
- link BR_Caster_Wheel_Link: geometry collision cylinder length=0.044 radius=0.05; visual mesh filename=package://robot_description/meshes/BR_Caster_Wheel_Link.STL
- link DL_Link: geometry collision cylinder length=0.05 radius=0.08; visual mesh filename=package://robot_description/meshes/DL_Link.STL
- link DR_Link: geometry collision cylinder length=0.05 radius=0.08; visual mesh filename=package://robot_description/meshes/DR_Link.STL
- link FL_Caster_Wheel_Link: geometry collision cylinder length=0.044 radius=0.05; visual mesh filename=package://robot_description/meshes/FL_Caster_Wheel_Link.STL
- link FR_Caster_Wheel_Link: geometry collision cylinder length=0.044 radius=0.05; visual mesh filename=package://robot_description/meshes/FR_Caster_Wheel_Link.STL
- link base_link: geometry collision box size=0.8 0.6 0.37; visual mesh filename=package://robot_description/meshes/base_body_visual.STL

File: robotics/robot_description/urdf/amr_real.urdf.xacro (robot description, xacro)
@@ -15,5 +15,5 @@
        =================================================================== -->
   <xacro:property name="wheel_radius"     value="0.080"/>   <!-- metres: measured from DR_Link/DL_Link.STL bounding box (was 0.060, wrong scale -> odom drift) -->
-  <xacro:property name="wheel_separation" value="0.5787"/>  <!-- from DL/DR joint origins (2 x 0.28935) -->
+  <xacro:property name="wheel_separation" value="0.5787"/>  <!-- CAD joint centres: 2 x 0.28935 m -->
   <xacro:property name="base_to_axle_z"   value="0.3305"/>  <!-- CAD: base_link height above wheel axle (DR/DL joint z = -0.3305) -->
   <!-- LiDAR + IMU mount points on base_link (EDIT to real positions) -->
@@ -74,4 +74,10 @@
       <max_angular_velocity>1.8</max_angular_velocity>
       <min_angular_velocity>-1.8</min_angular_velocity>
+      <!-- Avoid an instantaneous wheel-speed step, which otherwise produces
+           a large initial slip and immediately corrupts wheel odometry. -->
+      <max_linear_acceleration>0.5</max_linear_acceleration>
+      <min_linear_acceleration>-0.5</min_linear_acceleration>
+      <max_angular_acceleration>1.5</max_angular_acceleration>
+      <min_angular_acceleration>-1.5</min_angular_acceleration>
     </plugin>
     <plugin filename="gz-sim-joint-state-publisher-system"
@@ -120,9 +126,16 @@
   </gazebo>
   <!-- ===================================================================
-       6. Zero-friction casters (passive: must not fight the drive)
+       6. Passive caster contact
+       Low rolling friction lets each wheel spin; higher lateral friction and
+       the caster trail rotate the swivel into the direction of travel.
        =================================================================== -->
-  <gazebo reference="FR_Caster_Wheel_Link"><mu1>0.0</mu1><mu2>0.0</mu2></gazebo>
-  <gazebo reference="FL_Caster_Wheel_Link"><mu1>0.0</mu1><mu2>0.0</mu2></gazebo>
-  <gazebo reference="BR_Caster_Wheel_Link"><mu1>0.0</mu1><mu2>0.0</mu2></gazebo>
-  <gazebo reference="BL_Caster_Wheel_Link"><mu1>0.0</mu1><mu2>0.0</mu2></gazebo>
+  <gazebo reference="FR_Caster_Wheel_Link"><mu1>0.1</mu1><mu2>0.2</mu2><fdir1>1 0 0</fdir1></gazebo>
+  <gazebo reference="FL_Caster_Wheel_Link"><mu1>0.1</mu1><mu2>0.2</mu2><fdir1>1 0 0</fdir1></gazebo>
+  <gazebo reference="BR_Caster_Wheel_Link"><mu1>0.1</mu1><mu2>0.2</mu2><fdir1>1 0 0</fdir1></gazebo>
+  <gazebo reference="BL_Caster_Wheel_Link"><mu1>0.1</mu1><mu2>0.2</mu2><fdir1>1 0 0</fdir1></gazebo>
+  <!-- Positive drive-wheel traction. Primitive cylinder collisions in the CAD
+       URDF provide a smooth rolling surface; these values prevent sustained
+       wheel slip without making differential-drive turning excessively stiff. -->
+  <gazebo reference="DR_Link"><mu1>3.0</mu1><mu2>3.0</mu2></gazebo>
+  <gazebo reference="DL_Link"><mu1>3.0</mu1><mu2>3.0</mu2></gazebo>
 </robot>
