Commit message: fixed the robot drifting problem

File: robotics/robot_description/urdf/amr_2lidar.urdf.xacro (robot description, xacro)
@@ -17,5 +17,5 @@
        =================================================================== -->
   <xacro:property name="wheel_radius"     value="0.080"/>   <!-- VERIFY: not derivable from the CAD export -->
-  <xacro:property name="wheel_separation" value="0.5787"/>  <!-- from DL/DR joint origins (2 x 0.289353) -->
+  <xacro:property name="wheel_separation" value="0.541"/>  <!-- from DL/DR joint origins (2 x 0.289353) -->
   <xacro:property name="base_to_axle_z"   value="0.3305"/>  <!-- NEW CAD: DL/DR joint z = -0.3305 (was 0.3505) -->
   <!-- IMU mount point on base_link -->

Commit message: added a working test camera to the robot urdf publishing a real image of the environment. will be testing docking with apriltags across the environment.

File: robotics/robot_description/urdf/amr_2lidar.urdf.xacro (robot description, xacro)
@@ -34,4 +34,14 @@
   <xacro:property name="lidar_samples"      value="360"/>
   <xacro:property name="lidar_update_rate"  value="10"/>
+  <!-- Front-facing RGB camera (for AprilTag / visual-dock detection).
+       Mounted at the front edge, facing +X (robot forward), above the
+       Lidar deck. VERIFY xyz against wherever the real camera ends up. -->
+  <xacro:property name="camera_xyz"          value="0.40 0.0 0.15"/>
+  <xacro:property name="camera_rpy"          value="0 0 0"/>
+  <xacro:property name="camera_topic"        value="camera/image_raw"/>
+  <xacro:property name="camera_width"        value="640"/>
+  <xacro:property name="camera_height"       value="480"/>
+  <xacro:property name="camera_update_rate"  value="30"/>
+  <xacro:property name="camera_horizontal_fov" value="1.089"/> <!-- ~62 deg -->
   <!-- ===================================================================
        1. Pull in the NEW CAD export (chassis + casters + drive wheels +
@@ -59,4 +69,23 @@
     <child  link="imu_link"/>
     <origin xyz="${imu_xyz}" rpy="0 0 0"/>
+  </joint>
+  <!-- ===================================================================
+       3b. Camera frame. camera_link follows REP-103 (X fwd, Y left, Z up)
+           for a sane mount pose; camera_optical_link rotates into the
+           optical convention (Z fwd, X right, Y down) that image_geometry
+           / apriltag_ros expect, and is what the sensor reports as its
+           gz_frame_id below.
+       =================================================================== -->
+  <link name="camera_link"/>
+  <joint name="camera_joint" type="fixed">
+    <parent link="base_link"/>
+    <child  link="camera_link"/>
+    <origin xyz="${camera_xyz}" rpy="${camera_rpy}"/>
+  </joint>
+  <link name="camera_optical_link"/>
+  <joint name="camera_optical_joint" type="fixed">
+    <parent link="camera_link"/>
+    <child  link="camera_optical_link"/>
+    <origin xyz="0 0 0" rpy="-1.5708 0 -1.5708"/>
   </joint>
   <!-- ===================================================================
@@ -169,4 +198,31 @@
   </gazebo>
   <!-- ===================================================================
+       6b. Camera sensor -> publishes ${camera_topic}/image + camera_info.
+           gz_frame_id points at the optical frame, not camera_link, so
+           downstream image consumers (apriltag_ros, image_proc) get poses
+           in the standard camera-optical convention without a re-rotation.
+       =================================================================== -->
+  <gazebo reference="camera_link">
+    <sensor name="camera" type="camera">
+      <topic>${camera_topic}</topic>
+      <gz_frame_id>camera_optical_link</gz_frame_id>
+      <update_rate>${camera_update_rate}</update_rate>
+      <always_on>true</always_on>
+      <visualize>true</visualize>
+      <camera>
+        <horizontal_fov>${camera_horizontal_fov}</horizontal_fov>
+        <image>
+          <width>${camera_width}</width>
+          <height>${camera_height}</height>
+          <format>R8G8B8</format>
+        </image>
+        <clip>
+          <near>0.05</near>
+          <far>30.0</far>
+        </clip>
+      </camera>
+    </sensor>
+  </gazebo>
+  <!-- ===================================================================
        7. Zero-friction casters (passive: must not fight the drive)
        =================================================================== -->

Commit message: Revert "added a working test camera to the robot urdf publishing a real image of the environment. will be testing docking with apriltags across the environment."
This reverts commit 447b38341720beef2a7b133ed0c9b6be2c51a965.

File: robotics/robot_description/urdf/amr_2lidar.urdf.xacro (robot description, xacro)
@@ -34,14 +34,4 @@
   <xacro:property name="lidar_samples"      value="360"/>
   <xacro:property name="lidar_update_rate"  value="10"/>
-  <!-- Front-facing RGB camera (for AprilTag / visual-dock detection).
-       Mounted at the front edge, facing +X (robot forward), above the
-       Lidar deck. VERIFY xyz against wherever the real camera ends up. -->
-  <xacro:property name="camera_xyz"          value="0.40 0.0 0.15"/>
-  <xacro:property name="camera_rpy"          value="0 0 0"/>
-  <xacro:property name="camera_topic"        value="camera/image_raw"/>
-  <xacro:property name="camera_width"        value="640"/>
-  <xacro:property name="camera_height"       value="480"/>
-  <xacro:property name="camera_update_rate"  value="30"/>
-  <xacro:property name="camera_horizontal_fov" value="1.089"/> <!-- ~62 deg -->
   <!-- ===================================================================
        1. Pull in the NEW CAD export (chassis + casters + drive wheels +
@@ -69,23 +59,4 @@
     <child  link="imu_link"/>
     <origin xyz="${imu_xyz}" rpy="0 0 0"/>
-  </joint>
-  <!-- ===================================================================
-       3b. Camera frame. camera_link follows REP-103 (X fwd, Y left, Z up)
-           for a sane mount pose; camera_optical_link rotates into the
-           optical convention (Z fwd, X right, Y down) that image_geometry
-           / apriltag_ros expect, and is what the sensor reports as its
-           gz_frame_id below.
-       =================================================================== -->
-  <link name="camera_link"/>
-  <joint name="camera_joint" type="fixed">
-    <parent link="base_link"/>
-    <child  link="camera_link"/>
-    <origin xyz="${camera_xyz}" rpy="${camera_rpy}"/>
-  </joint>
-  <link name="camera_optical_link"/>
-  <joint name="camera_optical_joint" type="fixed">
-    <parent link="camera_link"/>
-    <child  link="camera_optical_link"/>
-    <origin xyz="0 0 0" rpy="-1.5708 0 -1.5708"/>
   </joint>
   <!-- ===================================================================
@@ -198,31 +169,4 @@
   </gazebo>
   <!-- ===================================================================
-       6b. Camera sensor -> publishes ${camera_topic}/image + camera_info.
-           gz_frame_id points at the optical frame, not camera_link, so
-           downstream image consumers (apriltag_ros, image_proc) get poses
-           in the standard camera-optical convention without a re-rotation.
-       =================================================================== -->
-  <gazebo reference="camera_link">
-    <sensor name="camera" type="camera">
-      <topic>${camera_topic}</topic>
-      <gz_frame_id>camera_optical_link</gz_frame_id>
-      <update_rate>${camera_update_rate}</update_rate>
-      <always_on>true</always_on>
-      <visualize>true</visualize>
-      <camera>
-        <horizontal_fov>${camera_horizontal_fov}</horizontal_fov>
-        <image>
-          <width>${camera_width}</width>
-          <height>${camera_height}</height>
-          <format>R8G8B8</format>
-        </image>
-        <clip>
-          <near>0.05</near>
-          <far>30.0</far>
-        </clip>
-      </camera>
-    </sensor>
-  </gazebo>
-  <!-- ===================================================================
        7. Zero-friction casters (passive: must not fight the drive)
        =================================================================== -->

Commit message: added the inspection module sensors to the robot description folder.

File: robotics/robot_description/urdf/amr_2lidar.urdf.xacro (robot description, xacro)
@@ -247,3 +247,69 @@
   <gazebo reference="BR_Caster_Wheel_Link"><mu1>0.0</mu1><mu2>0.0</mu2></gazebo>
   <gazebo reference="BL_Caster_Wheel_Link"><mu1>0.0</mu1><mu2>0.0</mu2></gazebo>
+  <!-- ==== INSPECTION MODULE (thermal camera + gas sensor) ==== -->
+  <link name="cameras_mount_Link">
+    <inertial>
+      <origin xyz="-0.040236 0.013428 -0.026709" rpy="0 0 0"/>
+      <mass value="0.14071"/>
+      <inertia ixx="5.798E-05" ixy="3.3384E-07" ixz="-1.7319E-07"
+               iyy="1.6986E-05" iyz="1.6883E-08" izz="5.5627E-05"/>
+    </inertial>
+    <visual>
+      <origin xyz="0 0 0" rpy="0 0 0"/>
+      <geometry><mesh filename="package://robot_description/meshes/cameras_mount_Link.STL"/></geometry>
+      <material name="inspection_mount_green"><color rgba="0 0.7451 0 1"/></material>
+    </visual>
+    <collision>
+      <origin xyz="0 0 0" rpy="0 0 0"/>
+      <geometry><mesh filename="package://robot_description/meshes/cameras_mount_Link.STL"/></geometry>
+    </collision>
+  </link>
+  <joint name="cameras_mount_joint" type="fixed">
+    <origin xyz="0.51252 -0.0115 0.13975" rpy="0 0.020136 0"/>
+    <parent link="base_link"/>
+    <child link="cameras_mount_Link"/>
+  </joint>
+  <link name="camera_thermal_Link">
+    <inertial>
+      <origin xyz="-0.025189 4.4462E-06 -7.318E-05" rpy="0 0 0"/>
+      <mass value="0.008096"/>
+      <inertia ixx="6.1294E-07" ixy="7.4569E-11" ixz="-1.4303E-09"
+               iyy="4.3511E-07" iyz="-4.9824E-11" izz="4.3599E-07"/>
+    </inertial>
+    <visual>
+      <origin xyz="0 0 0" rpy="0 0 0"/>
+      <geometry><mesh filename="package://robot_description/meshes/camera_thermal_Link.STL"/></geometry>
+      <material name="inspection_thermal_grey"><color rgba="0.89412 0.89412 0.89412 1"/></material>
+    </visual>
+    <collision>
+      <origin xyz="0 0 0" rpy="0 0 0"/>
+      <geometry><mesh filename="package://robot_description/meshes/camera_thermal_Link.STL"/></geometry>
+    </collision>
+  </link>
+  <joint name="camera_thermal_joint" type="fixed">
+    <origin xyz="0.018405 0.0095726 0.02568" rpy="0 0 0"/>
+    <parent link="cameras_mount_Link"/>
+    <child link="camera_thermal_Link"/>
+  </joint>
+  <link name="GAZ_sensor_Link">
+    <inertial>
+      <origin xyz="0 0 0" rpy="0 0 0"/>
+      <mass value="0.001"/>
+      <inertia ixx="1e-6" ixy="0" ixz="0" iyy="1e-6" iyz="0" izz="1e-6"/>
+    </inertial>
+    <visual>
+      <origin xyz="0 0 0" rpy="0 0 0"/>
+      <geometry><mesh filename="package://robot_description/meshes/GAZ_sensor_Link.STL"/></geometry>
+      <material name="inspection_gas_white"><color rgba="1 1 1 1"/></material>
+    </visual>
+    <collision>
+      <origin xyz="0 0 0" rpy="0 0 0"/>
+      <geometry><mesh filename="package://robot_description/meshes/GAZ_sensor_Link.STL"/></geometry>
+    </collision>
+  </link>
+  <joint name="GAZ_sensor_Joint" type="fixed">
+    <origin xyz="0.23945 -0.30074 -0.235" rpy="0 0 0"/>
+    <parent link="base_link"/>
+    <child link="GAZ_sensor_Link"/>
+  </joint>
 </robot>

Commit message: reconfigured the camera link to match the new camera mount in the updated URDF .

File: robotics/robot_description/urdf/amr_2lidar.urdf.xacro (robot description, xacro)
@@ -35,7 +35,10 @@
   <xacro:property name="lidar_update_rate"  value="10"/>
   <!-- Front-facing RGB camera (for AprilTag / visual-dock detection).
-       Mounted at the front edge, facing +X (robot forward), above the
-       Lidar deck. VERIFY xyz against wherever the real camera ends up. -->
-  <xacro:property name="camera_xyz"          value="0.40 0.0 0.15"/>
+       Mounted on the real cameras_mount_Link bracket (see INSPECTION MODULE
+       below), beside camera_thermal_Link, rather than floating off
+       base_link at a guessed position. xyz/rpy are relative to
+       cameras_mount_Link's own frame. VERIFY against the actual bracket
+       once the real camera is fitted. -->
+  <xacro:property name="camera_xyz"          value="0.0 -0.05 0.02"/>
   <xacro:property name="camera_rpy"          value="0 0 0"/>
   <xacro:property name="camera_topic"        value="camera/image_raw"/>
@@ -80,4 +83,8 @@
            body can't be welded by the physics engine - it just drifts
            free instead of staying mounted.
+           Parented to cameras_mount_Link (defined below, under INSPECTION
+           MODULE) rather than base_link directly - that's the real mount
+           bracket your camera actually lives on, alongside
+           camera_thermal_Link.
        =================================================================== -->
   <link name="camera_link">
@@ -89,5 +96,5 @@
   </link>
   <joint name="camera_joint" type="fixed">
-    <parent link="base_link"/>
+    <parent link="cameras_mount_Link"/>
     <child  link="camera_link"/>
     <origin xyz="${camera_xyz}" rpy="${camera_rpy}"/>
