Commit message: Refine AMR-X visual finishes

File: robotics/robot_description/urdf/AMR-2Lidar-Link.urdf (robot description, URDF)
Before this commit: robot AMR-2Lidar-Link, 13 links, 12 joints
Links:
- link base_link: geometry collision mesh filename=package://robot_description/meshes/base_link.STL; visual mesh filename=package://robot_description/meshes/base_body_visual.STL

File: robotics/robot_description/urdf/amr_2lidar.urdf.xacro (robot description, xacro)
@@ -265,5 +265,5 @@
       <origin xyz="0 0 0" rpy="0 0 0"/>
       <geometry><mesh filename="package://robot_description/meshes/cameras_mount_Link.STL"/></geometry>
-      <material name="inspection_mount_green"><color rgba="0 0.7451 0 1"/></material>
+      <material name="amrx_medical_teal"><color rgba="0 0.38 0.46 1"/></material>
     </visual>
     <collision>
@@ -287,5 +287,5 @@
       <origin xyz="0 0 0" rpy="0 0 0"/>
       <geometry><mesh filename="package://robot_description/meshes/camera_thermal_Link.STL"/></geometry>
-      <material name="inspection_thermal_grey"><color rgba="0.89412 0.89412 0.89412 1"/></material>
+      <material name="amrx_sensor_graphite"><color rgba="0.06 0.08 0.10 1"/></material>
     </visual>
     <collision>
@@ -308,5 +308,5 @@
       <origin xyz="0 0 0" rpy="0 0 0"/>
       <geometry><mesh filename="package://robot_description/meshes/GAZ_sensor_Link.STL"/></geometry>
-      <material name="inspection_gas_white"><color rgba="1 1 1 1"/></material>
+      <material name="amrx_porcelain_white"><color rgba="0.82 0.86 0.88 1"/></material>
     </visual>
     <collision>

File: robotics/robot_description/urdf/amr_inspection.urdf.xacro (robot description, xacro)
@@ -37,6 +37,6 @@
         <mesh filename="package://robot_description/meshes/cameras_mount_Link.STL"/>
       </geometry>
-      <material name="inspection_mount_green">
-        <color rgba="0 0.7451 0 1"/>
+      <material name="amrx_medical_teal">
+        <color rgba="0 0.38 0.46 1"/>
       </material>
     </visual>
@@ -66,6 +66,6 @@
         <mesh filename="package://robot_description/meshes/camera_thermal_Link.STL"/>
       </geometry>
-      <material name="inspection_thermal_grey">
-        <color rgba="0.89412 0.89412 0.89412 1"/>
+      <material name="amrx_sensor_graphite">
+        <color rgba="0.06 0.08 0.10 1"/>
       </material>
     </visual>
@@ -94,6 +94,6 @@
         <mesh filename="package://robot_description/meshes/GAZ_sensor_Link.STL"/>
       </geometry>
-      <material name="inspection_gas_white">
-        <color rgba="1 1 1 1"/>
+      <material name="amrx_porcelain_white">
+        <color rgba="0.82 0.86 0.88 1"/>
       </material>
     </visual>

File: robotics/robot_description/urdf/amr_with_arm.xacro (robot description, xacro)
@@ -105,6 +105,6 @@
         <box size="0.105 0.14 0.008"/>
       </geometry>
-      <material name="dark_grey">
-        <color rgba="1 0 0 1.0"/>
+      <material name="amrx_graphite_hardware">
+        <color rgba="0.16 0.19 0.22 1"/>
       </material>
     </visual>
