Commit message: Implement arm description, control, and MoveIt config with working Gazebo simulation

File: robotics/arm_description/urdf/arm_gazebo.xacro (robot description, xacro)
@@ -1 +1,15 @@
-# TODO(team): Gazebo Fortress ros2_control tags for arm joints
+<?xml version="1.0" ?>
+<robot xmlns:xacro="http://wiki.ros.org/xacro">
+    <xacro:macro name="load_gazebo_sim_ros2_control_plugin" params="robot_name use_gazebo">
+        <xacro:if value="${use_gazebo}">
+            <gazebo>
+                <plugin filename="gz_ros2_control-system" name="gz_ros2_control::GazeboSimROS2ControlPlugin">
+                    <parameters>$(find arm_control)/config/arm_controllers.yaml</parameters>
+                    <ros>
+                        <remapping>/controller_manager/robot_description:=/robot_description</remapping>
+                    </ros>
+                </plugin>
+            </gazebo>
+        </xacro:if>
+    </xacro:macro>
+</robot>

File: robotics/arm_description/urdf/arm_module.xacro (robot description, xacro)
@@ -1 +1,52 @@
-# TODO(team): top-level arm module xacro: mount to base + include both arms
+<?xml version="1.0"?>
+<robot xmlns:xacro="http://www.ros.org/wiki/xacro" name="arm_module">
+    <xacro:arg name="robot_name" default="mycobot_280"/>
+    <xacro:arg name="add_world" default="true"/>
+    <xacro:arg name="base_link" default="base_link"/>
+    <xacro:arg name="base_type" default="g_shape"/>
+    <xacro:arg name="flange_link" default="link6_flange"/>
+    <xacro:arg name="gripper_type" default="gripper"/>
+    <xacro:arg name="prefix" default=""/>
+    <xacro:arg name="use_camera" default="false"/>
+    <xacro:arg name="use_gazebo" default="false"/>
+    <xacro:arg name="use_gripper" default="true"/>
+    <xacro:arg name="add_world" default="true"/>
+    <xacro:if value="$(arg add_world)">
+    <link name="world"/>
+    <joint name="$(arg prefix)virtual_joint" type="fixed">
+        <parent link="world"/>
+        <child link="$(arg prefix)$(arg base_link)"/>
+        <origin xyz="0 0 0" rpy="0 0 0"/>
+    </joint>
+    </xacro:if>
+    <xacro:include filename="$(find arm_description)/urdf/single_arm.xacro"/>
+    <xacro:g_shape_base
+        base_link="$(arg base_link)"
+        prefix="$(arg prefix)"/>
+    <xacro:single_arm
+      base_link="$(arg base_link)"
+      flange_link="$(arg flange_link)"
+      prefix="$(arg prefix)">
+      <origin xyz="0 0 0" rpy="0 0 0"/>
+    </xacro:single_arm>
+    <xacro:if value="$(arg use_gripper)">
+        <xacro:property name="current_gripper" value="$(arg gripper_type)"/>
+        <xacro:if value="${current_gripper == 'gripper'}">
+            <xacro:include filename="$(find arm_description)/urdf/gripper.xacro"/>
+            <xacro:gripper
+                parent="$(arg flange_link)"
+                prefix="$(arg prefix)">
+                <origin xyz="0 0 0.034" rpy="1.579 0 0"/>
+            </xacro:gripper>
+        </xacro:if>
+    </xacro:if>
+    <xacro:include filename="$(find arm_description)/urdf/arm_gazebo.xacro"/>
+        <xacro:load_gazebo_sim_ros2_control_plugin
+        robot_name="$(arg robot_name)"
+        use_gazebo="$(arg use_gazebo)"/>
+        <xacro:include filename="$(find arm_description)/urdf/arm_control.xacro"/>
+        <xacro:arm_ros2_control
+        prefix="$(arg prefix)"
+        flange_link="$(arg flange_link)"
+        use_gazebo="$(arg use_gazebo)"/>
+</robot>

File: robotics/arm_description/urdf/gripper.xacro (robot description, xacro)
@@ -1 +1,202 @@
-# TODO(team): gripper / end-effector macro
+<?xml version="1.0"?>
+<robot xmlns:xacro="http://www.ros.org/wiki/xacro">
+  <xacro:property name="joint_effort" value="56.0"/>
+  <xacro:property name="joint_velocity" value="2.792527"/>
+  <xacro:property name="joint_damping" value="0.0"/>
+  <xacro:property name="joint_friction" value="0.0"/>
+  <xacro:property name="gripper_link_mass" value="0.007"/>
+  <xacro:property name="gripper_link_ixx" value="1e-6"/>
+  <xacro:property name="gripper_link_iyy" value="1e-6"/>
+  <xacro:property name="gripper_link_izz" value="1e-6"/>
+  <xacro:macro name="gripper_link_inertial">
+    <inertial>
+      <origin xyz="0 0 0.0" rpy="0 0 0"/>
+      <mass value="${gripper_link_mass}"/>
+      <inertia
+        ixx="${gripper_link_ixx}" ixy="0.0" ixz="0.0"
+        iyy="${gripper_link_iyy}" iyz="0.0"
+        izz="${gripper_link_izz}"/>
+    </inertial>
+  </xacro:macro>
+  <xacro:macro name="gripper" params="parent prefix *origin">
+    <link name="${prefix}gripper_base">
+      <inertial>
+        <origin xyz="0 0 0.0" rpy="0 0 0"/>
+        <mass value="0.07"/>
+        <inertia
+          ixx="0.000010725" ixy="0.0" ixz="0.0"
+          iyy="0.000014392" iyz="0.0"
+          izz="0.000018517"/>
+      </inertial>
+      <visual>
+        <geometry>
+          <mesh filename="file://$(find arm_description)/meshes/adaptive_gripper/visual/gripper_base.dae"/>
+        </geometry>
+        <origin xyz="0.0 0.0 -0.012" rpy="0 0 0"/>
+      </visual>
+      <collision>
+        <geometry>
+          <box size="0.065 0.025 0.025"/>
+        </geometry>
+        <origin xyz="0.0 0.0 0.0" rpy="0 0 0"/>
+      </collision>
+    </link>
+    <joint name="${prefix}${parent}_to_${prefix}gripper_base" type="fixed">
+      <parent link="${prefix}${parent}"/>
+      <child link="${prefix}gripper_base"/>
+      <xacro:insert_block name="origin"/>
+    </joint>
+    <link name="${prefix}gripper_left1">
+      <xacro:gripper_link_inertial/>
+      <visual>
+        <geometry>
+          <mesh filename="file://$(find arm_description)/meshes/adaptive_gripper/visual/gripper_left1.dae"/>
+        </geometry>
+        <origin xyz="0.039 -0.0133 -0.012" rpy="0 0 0"/>
+      </visual>
+      <collision>
+        <geometry>
+          <box size="0.013 0.02 0.015"/>
+        </geometry>
+        <origin xyz="0.013 0.042 -0.010" rpy="0 0 0"/>
+      </collision>
+    </link>
+    <link name="${prefix}gripper_left2">
+      <xacro:gripper_link_inertial/>
+      <visual>
+        <geometry>
+          <mesh filename="file://$(find arm_description)/meshes/adaptive_gripper/visual/gripper_left2.dae"/>
+        </geometry>
+        <origin xyz="0.005 -0.0195 -0.012" rpy="0 0 0"/>
+      </visual>
+      <collision>
+        <geometry>
+          <box size="0.02 0.02 0.02"/>
+        </geometry>
+        <origin xyz="-0.025 0.0 -0.010" rpy="0 0 0"/>
+      </collision>
+    </link>
+    <link name="${prefix}gripper_left3">
+      <xacro:gripper_link_inertial/>
+      <visual>
+        <geometry>
+          <mesh filename="file://$(find arm_description)/meshes/adaptive_gripper/visual/gripper_left3.dae"/>
+        </geometry>
+        <origin xyz="0.012 0.0025 -0.012" rpy="0 0 0"/>
+      </visual>
+      <collision>
+        <geometry>
+          <box size="0.01 0.01 0.01"/>
+        </geometry>
+        <origin xyz="-0.014 0.005 0.005" rpy="0 0 0"/>
+      </collision>
+    </link>
+    <link name="${prefix}gripper_right1">
+      <xacro:gripper_link_inertial/>
+      <visual>
+        <geometry>
+          <mesh filename="file://$(find arm_description)/meshes/adaptive_gripper/visual/gripper_right1.dae"/>
+        </geometry>
+        <origin xyz="-0.039 -0.0133 -0.012" rpy="0 0 0"/>
+      </visual>
+      <collision>
+        <geometry>
+          <box size="0.013 0.02 0.015"/>
+        </geometry>
+        <origin xyz="-0.013 0.042 -0.010" rpy="0 0 0"/>
+      </collision>
+    </link>
+    <link name="${prefix}gripper_right2">
+      <xacro:gripper_link_inertial/>
+      <visual>
+        <geometry>
+          <mesh filename="file://$(find arm_description)/meshes/adaptive_gripper/visual/gripper_right2.dae"/>
+        </geometry>
+        <origin xyz="-0.005 -0.0195 -0.012" rpy="0 0 0"/>
+      </visual>
+      <collision>
+        <geometry>
+          <box size="0.02 0.02 0.02"/>
+        </geometry>
+        <origin xyz="0.025 0.0 -0.010" rpy="0 0 0"/>
+      </collision>
+    </link>
+    <link name="${prefix}gripper_right3">
+      <xacro:gripper_link_inertial/>
+      <visual>
+        <geometry>
+          <mesh filename="file://$(find arm_description)/meshes/adaptive_gripper/visual/gripper_right3.dae"/>
+        </geometry>
+        <origin xyz="-0.012 0.0025 -0.012" rpy="0 0 0"/>
+      </visual>
+      <collision>
+        <geometry>
+          <box size="0.01 0.01 0.01"/>
+        </geometry>
+        <origin xyz="0.014 0.005 0.005" rpy="0 0 0"/>
+      </collision>
+    </link>
+    <joint name="${prefix}gripper_controller" type="revolute">
+      <axis xyz="0 0 1"/>
+      <limit effort="${joint_effort}" lower="-0.7" upper="0.15" velocity="${joint_velocity}"/>
+      <parent link="${prefix}gripper_base"/>
+      <child link="${prefix}gripper_left3"/>
+      <origin xyz="-0.012 0.005 0" rpy="0 0 0"/>
+      <dynamics damping="${joint_damping}" friction="${joint_friction}"/>
+    </joint>
+    <joint name="${prefix}gripper_base_to_${prefix}gripper_left2" type="revolute">
+      <axis xyz="0 0 1"/>
+      <limit effort="${joint_effort}" lower="-0.8" upper="0.5" velocity="${joint_velocity}"/>
+      <parent link="${prefix}gripper_base"/>
+      <child link="${prefix}gripper_left2"/>
+      <origin xyz="-0.005 0.027 0" rpy="0 0 0"/>
+      <mimic joint="${prefix}gripper_controller" multiplier="1.0" offset="0"/>
+      <dynamics damping="${joint_damping}" friction="${joint_friction}"/>
+    </joint>
+    <joint name="${prefix}gripper_left3_to_${prefix}gripper_left1" type="revolute">
+      <axis xyz="0 0 1"/>
+      <limit effort="${joint_effort}" lower="-0.5" upper="0.5" velocity="${joint_velocity}"/>
+      <parent link="${prefix}gripper_left3"/>
+      <child link="${prefix}gripper_left1"/>
+      <origin xyz="-0.027 0.016 0" rpy="0 0 0"/>
+      <mimic joint="${prefix}gripper_controller" multiplier="-1.0" offset="0"/>
+      <dynamics damping="${joint_damping}" friction="${joint_friction}"/>
+    </joint>
+    <joint name="${prefix}gripper_base_to_${prefix}gripper_right3" type="revolute">
+      <axis xyz="0 0 1"/>
+      <limit effort="${joint_effort}" lower="-0.15" upper="0.7" velocity="${joint_velocity}"/>
+      <parent link="${prefix}gripper_base"/>
+      <child link="${prefix}gripper_right3"/>
+      <origin xyz="0.012 0.005 0" rpy="0 0 0"/>
+      <mimic joint="${prefix}gripper_controller" multiplier="-1.0" offset="0"/>
+      <dynamics damping="${joint_damping}" friction="${joint_friction}"/>
+    </joint>
+    <joint name="${prefix}gripper_base_to_${prefix}gripper_right2" type="revolute">
+      <axis xyz="0 0 1"/>
+      <limit effort="${joint_effort}" lower="-0.5" upper="0.8" velocity="${joint_velocity}"/>
+      <parent link="${prefix}gripper_base"/>
+      <child link="${prefix}gripper_right2"/>
+      <origin xyz="0.005 0.027 0" rpy="0 0 0"/>
+      <mimic joint="${prefix}gripper_controller" multiplier="-1.0" offset="0"/>
+      <dynamics damping="${joint_damping}" friction="${joint_friction}"/>
+    </joint>
+    <joint name="${prefix}gripper_right3_to_${prefix}gripper_right1" type="revolute">
+      <axis xyz="0 0 1"/>
+      <limit effort="${joint_effort}" lower="-0.5" upper="0.5" velocity="${joint_velocity}"/>
+      <parent link="${prefix}gripper_right3"/>
+      <child link="${prefix}gripper_right1"/>
+      <origin xyz="0.027 0.016 0" rpy="0 0 0"/>
+      <mimic joint="${prefix}gripper_controller" multiplier="1.0" offset="0"/>
+      <dynamics damping="${joint_damping}" friction="${joint_friction}"/>
+    </joint>
+    <gazebo reference="${prefix}gripper_base">
+      <visual>
+        <material>
+          <ambient>1 1 1 1</ambient>
+          <diffuse>1 1 1 1</diffuse>
+          <specular>1 1 1 1</specular>
+        </material>
+      </visual>
+    </gazebo>
+  </xacro:macro>
+</robot>

File: robotics/arm_description/urdf/single_arm.xacro (robot description, xacro)
@@ -1 +1,235 @@
-# TODO(team): single reusable arm macro, instantiated left + right
+<?xml version="1.0"?>
+<robot xmlns:xacro="http://www.ros.org/wiki/xacro">
+  <xacro:property name="joint_effort" value="56.0"/>
+  <xacro:property name="joint_velocity" value="2.792527"/>
+  <xacro:property name="joint_damping" value="0.0"/>
+  <xacro:property name="joint_friction" value="0.0"/>
+  <xacro:property name="link1_mass" value="0.12"/>
+  <xacro:property name="link2_mass" value="0.19"/>
+  <xacro:property name="link3_mass" value="0.16"/>
+  <xacro:property name="link4_mass" value="0.124"/>
+  <xacro:property name="link5_mass" value="0.11"/>
+  <xacro:property name="link6_mass" value="0.0739"/>
+  <xacro:property name="flange_mass" value="0.035"/>
+  <xacro:macro name="link_inertial" params="mass ixx iyy izz">
+    <inertial>
+      <origin xyz="0 0 0.0" rpy="0 0 0"/>
+      <mass value="${mass}"/>
+      <inertia
+        ixx="${ixx}" ixy="0.0" ixz="0.0"
+        iyy="${iyy}" iyz="0.0"
+        izz="${izz}"/>
+    </inertial>
+  </xacro:macro>
+  <xacro:macro name="material_visual" params="ref_link ambient diffuse specular">
+    <gazebo reference="${ref_link}">
+      <visual>
+        <material>
+          <ambient>${ambient}</ambient>
+          <diffuse>${diffuse}</diffuse>
+          <specular>${specular}</specular>
+        </material>
+      </visual>
+    </gazebo>
+  </xacro:macro>
+  <xacro:macro name="g_shape_base" params="base_link prefix">
+    <link name="${prefix}${base_link}">
+      <inertial>
+        <origin xyz="0 0 0.0" rpy="0 0 0"/>
+        <mass value="0.33"/>
+        <inertia
+          ixx="0.000784" ixy="0.0" ixz="0.0"
+          iyy="0.000867" iyz="0.0"
+          izz="0.001598"/>
+      </inertial>
+      <visual>
+        <geometry>
+          <mesh filename="file://$(find arm_description)/meshes/g_shape_base_v2_0/visual/base_link.dae"/>
+        </geometry>
+        <origin xyz="0.0 0 -0.03" rpy="0 0 ${pi/2}"/>
+      </visual>
+      <collision>
+        <geometry>
+          <box size="0.105 0.14 0.02"/>
+        </geometry>
+        <origin xyz="0.0 0.0 -0.015" rpy="0 0 0"/>
+      </collision>
+    </link>
+    <gazebo reference="${prefix}${base_link}">
+      <visual>
+        <material>
+          <ambient>0.5 0.5 0.5 1</ambient>
+          <diffuse>0.5 0.5 0.5 1</diffuse>
+          <specular>0.5 0.5 0.5 1</specular>
+        </material>
+      </visual>
+    </gazebo>
+  </xacro:macro>
+  <xacro:macro name="single_arm" params="base_link flange_link prefix *origin">
+    <link name="${prefix}link1">
+      <xacro:link_inertial mass="${link1_mass}" ixx="0.000148" iyy="0.000148" izz="0.000096"/>
+      <visual>
+        <geometry>
+          <mesh filename="file://$(find arm_description)/meshes/mycobot_280/visual/link1.dae"/>
+        </geometry>
+        <origin xyz="0.0 0 0" rpy="0 0 ${-pi/2}"/>
+      </visual>
+      <collision>
+        <geometry>
+          <box size="0.08 0.12 0.075"/>
+        </geometry>
+        <origin xyz="0.0 -0.01 0.034" rpy="0 0 0"/>
+      </collision>
+    </link>
+    <link name="${prefix}link2">
+      <xacro:link_inertial mass="${link2_mass}" ixx="0.000148" iyy="0.000148" izz="0.000096"/>
+      <visual>
+        <geometry>
+          <mesh filename="file://$(find arm_description)/meshes/mycobot_280/visual/link2.dae"/>
+        </geometry>
+        <origin xyz="0.0 0 -0.06096" rpy="0 0 ${-pi/2}"/>
+      </visual>
+      <collision>
+        <geometry>
+          <cylinder radius="0.025" length="0.085"/>
+        </geometry>
+        <origin xyz="0.0 0 -0.02" rpy="0 0 ${-pi/2}"/>
+      </collision>
+    </link>
+    <link name="${prefix}link3">
+      <xacro:link_inertial mass="${link3_mass}" ixx="0.000148" iyy="0.000148" izz="0.000096"/>
+      <visual>
+        <geometry>
+          <mesh filename="file://$(find arm_description)/meshes/mycobot_280/visual/link3.dae"/>
+        </geometry>
+        <origin xyz="0.0 0 0.03256" rpy="0 ${-pi/2} 0"/>
+      </visual>
+      <collision>
+        <geometry>
+          <cylinder radius="0.025" length="0.15"/>
+        </geometry>
+        <origin xyz="-0.058 0 0.059" rpy="0 ${-pi/2} 0"/>
+      </collision>
+    </link>
+    <link name="${prefix}link4">
+      <xacro:link_inertial mass="${link4_mass}" ixx="0.000103" iyy="0.000103" izz="0.000096"/>
+      <visual>
+        <geometry>
+          <mesh filename="file://$(find arm_description)/meshes/mycobot_280/visual/link4.dae"/>
+        </geometry>
+        <origin xyz="0.0 0 0.03056" rpy="0 ${-pi/2} 0"/>
+      </visual>
+      <collision>
+        <geometry>
+          <cylinder radius="0.025" length="0.125"/>
+        </geometry>
+        <origin xyz="-0.05 0 0.0" rpy="0 ${-pi/2} 0"/>
+      </collision>
+    </link>
+    <link name="${prefix}link5">
+      <xacro:link_inertial mass="${link5_mass}" ixx="0.000103" iyy="0.000103" izz="0.000096"/>
+      <visual>
+        <geometry>
+          <mesh filename="file://$(find arm_description)/meshes/mycobot_280/visual/link5.dae"/>
+        </geometry>
+        <origin xyz="0.0 0 -0.03356" rpy="${-pi/2} 0 0"/>
+      </visual>
+      <collision>
+        <geometry>
+          <box size="0.03 0.035 0.05"/>
+        </geometry>
+        <origin xyz="0.0 0 -0.005" rpy="0 0.0 0"/>
+      </collision>
+    </link>
+    <link name="${prefix}link6">
+      <xacro:link_inertial mass="${link6_mass}" ixx="0.00006649" iyy="0.00006649" izz="0.000096"/>
+      <visual>
+        <geometry>
+          <mesh filename="file://$(find arm_description)/meshes/mycobot_280/visual/link6.dae"/>
+        </geometry>
+        <origin xyz="0 0.00 -0.038" rpy="0 0 0"/>
+      </visual>
+      <collision>
+        <geometry>
+          <cylinder radius="0.025" length="0.06"/>
+        </geometry>
+        <origin xyz="0 0.00 0.0" rpy="${-pi/2} 0 0"/>
+      </collision>
+    </link>
+    <link name="${prefix}${flange_link}">
+      <xacro:link_inertial mass="${flange_mass}" ixx="0.0000149" iyy="0.0000149" izz="0.0000196"/>
+      <visual>
+        <geometry>
+          <mesh filename="file://$(find arm_description)/meshes/mycobot_280/visual/link7.dae"/>
+        </geometry>
+        <origin xyz="0.0 0 -0.012" rpy="0 0 0"/>
+      </visual>
+      <collision>
+        <geometry>
+          <cylinder radius="0.02" length="0.02"/>
+        </geometry>
+        <origin xyz="0 0.00 0.0" rpy="0 0 0"/>
+      </collision>
+    </link>
+    <joint name="${prefix}${base_link}_to_${prefix}link1" type="fixed">
+      <parent link="${prefix}${base_link}"/>
+      <child link="${prefix}link1"/>
+      <xacro:insert_block name="origin"/>
+    </joint>
+    <joint name="${prefix}link1_to_${prefix}link2" type="revolute">
+      <axis xyz="0 0 1"/>
+      <limit effort="${joint_effort}" lower="-2.879793" upper="2.879793" velocity="${joint_velocity}"/>
+      <parent link="${prefix}link1"/>
+      <child link="${prefix}link2"/>
+      <origin xyz="0 0 0.13156" rpy="0 0 ${pi/2}"/>
+      <dynamics damping="${joint_damping}" friction="${joint_friction}"/>
+    </joint>
+    <joint name="${prefix}link2_to_${prefix}link3" type="revolute">
+      <axis xyz="0 0 1"/>
+      <limit effort="${joint_effort}" lower="-2.879793" upper="2.879793" velocity="${joint_velocity}"/>
+      <parent link="${prefix}link2"/>
+      <child link="${prefix}link3"/>
+      <origin xyz="0 0 -0.001" rpy="0 ${pi/2} ${-pi/2}"/>
+      <dynamics damping="${joint_damping}" friction="${joint_friction}"/>
+    </joint>
+    <joint name="${prefix}link3_to_${prefix}link4" type="revolute">
+      <axis xyz="0 0 1"/>
+      <limit effort="${joint_effort}" lower="-2.879793" upper="2.879793" velocity="${joint_velocity}"/>
+      <parent link="${prefix}link3"/>
+      <child link="${prefix}link4"/>
+      <origin xyz="-0.1104 0 0" rpy="0 0 0"/>
+      <dynamics damping="${joint_damping}" friction="${joint_friction}"/>
+    </joint>
+    <joint name="${prefix}link4_to_${prefix}link5" type="revolute">
+      <axis xyz="0 0 1"/>
+      <limit effort="${joint_effort}" lower="-2.879793" upper="2.879793" velocity="${joint_velocity}"/>
+      <parent link="${prefix}link4"/>
+      <child link="${prefix}link5"/>
+      <origin xyz="-0.096 0 0.06062" rpy="0 0 ${-pi/2}"/>
+      <dynamics damping="${joint_damping}" friction="${joint_friction}"/>
+    </joint>
+    <joint name="${prefix}link5_to_${prefix}link6" type="revolute">
+      <axis xyz="0 0 1"/>
+      <limit effort="${joint_effort}" lower="-2.879793" upper="2.879793" velocity="${joint_velocity}"/>
+      <parent link="${prefix}link5"/>
+      <child link="${prefix}link6"/>
+      <origin xyz="0 -0.07318 0" rpy="${pi/2} ${-pi/2} 0"/>
+      <dynamics damping="${joint_damping}" friction="${joint_friction}"/>
+    </joint>
+    <joint name="${prefix}link6_to_${prefix}${flange_link}" type="revolute">
+      <axis xyz="0 0 1"/>
+      <limit effort="${joint_effort}" lower="-3.05" upper="3.05" velocity="${joint_velocity}"/>
+      <parent link="${prefix}link6"/>
+      <child link="${prefix}${flange_link}"/>
+      <origin xyz="0 0.0456 0" rpy="${-pi/2} 0 0"/>
+      <dynamics damping="${joint_damping}" friction="${joint_friction}"/>
+    </joint>
+    <xacro:material_visual ref_link="${prefix}link1" ambient="0.5 0.5 0.5 1" diffuse="0.5 0.5 0.5 1" specular="0.5 0.5 0.5 1"/>
+    <xacro:material_visual ref_link="${prefix}link2" ambient="1 1 1 1" diffuse="1 1 1 1" specular="1 1 1 1"/>
+    <xacro:material_visual ref_link="${prefix}link3" ambient="1 1 1 1" diffuse="1 1 1 1" specular="1 1 1 1"/>
+    <xacro:material_visual ref_link="${prefix}link4" ambient="1 1 1 1" diffuse="1 1 1 1" specular="1 1 1 1"/>
+    <xacro:material_visual ref_link="${prefix}link5" ambient="1 1 1 1" diffuse="1 1 1 1" specular="1 1 1 1"/>
+    <xacro:material_visual ref_link="${prefix}link6" ambient="1 1 1 1" diffuse="1 1 1 1" specular="1 1 1 1"/>
+    <xacro:material_visual ref_link="${prefix}${flange_link}" ambient="0.5 0.5 0.5 1" diffuse="0.5 0.5 0.5 1" specular="0.5 0.5 0.5 1"/>
+  </xacro:macro>
+</robot>
