Commit message: fix: add world link, fix mesh paths, add joint limits

File: robotics/dual_arm_description/urdf/dual_arm.urdf (robot description, URDF)
Before this commit: robot dual_arm, 18 links, 17 joints
Links:
- added link world
- link base_link: geometry collision mesh filename=file:///home/ubuntu/robot_ws/install/dual_arm_description/s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; visual mesh filename=file:///home/ubuntu/robot_ws/install/dual_arm_description/s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
- link pinion: geometry collision mesh filename=file:///home/ubuntu/robot_ws/install/dual_arm_description/s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; visual mesh filename=file:///home/ubuntu/robot_ws/install/dual_arm_description/s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
- link rack: geometry collision mesh filename=file:///home/ubuntu/robot_ws/install/dual_arm_description/s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; visual mesh filename=file:///home/ubuntu/robot_ws/install/dual_arm_description/s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
- link robot_base: geometry collision mesh filename=file:///home/ubuntu/robot_ws/install/dual_arm_description/s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; visual mesh filename=file:///home/ubuntu/robot_ws/install/dual_arm_description/s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
- link shoulderR_1: geometry collision mesh filename=file:///home/ubuntu/robot_ws/install/dual_arm_description/s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; visual mesh filename=file:///home/ubuntu/robot_ws/install/dual_arm_description/s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
- link shoulderR_2: geometry collision mesh filename=file:///home/ubuntu/robot_ws/install/dual_arm_description/s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; visual mesh filename=file:///home/ubuntu/robot_ws/install/dual_arm_description/s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
- link shoulderR_3: geometry collision mesh filename=file:///home/ubuntu/robot_ws/install/dual_arm_description/s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; visual mesh filename=file:///home/ubuntu/robot_ws/install/dual_arm_description/s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
- link shoulderR_4: geometry collision mesh filename=file:///home/ubuntu/robot_ws/install/dual_arm_description/s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; visual mesh filename=file:///home/ubuntu/robot_ws/install/dual_arm_description/s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
- link shoulderR_5: geometry collision mesh filename=file:///home/ubuntu/robot_ws/install/dual_arm_description/s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; visual mesh filename=file:///home/ubuntu/robot_ws/install/dual_arm_description/s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
- link shoulderR_6: geometry collision mesh filename=file:///home/ubuntu/robot_ws/install/dual_arm_description/s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; visual mesh filename=file:///home/ubuntu/robot_ws/install/dual_arm_description/s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
- link shoulder_1: geometry collision mesh filename=file:///home/ubuntu/robot_ws/install/dual_arm_description/s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; visual mesh filename=file:///home/ubuntu/robot_ws/install/dual_arm_description/s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
- link shoulder_2: geometry collision mesh filename=file:///home/ubuntu/robot_ws/install/dual_arm_description/s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; visual mesh filename=file:///home/ubuntu/robot_ws/install/dual_arm_description/s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
- link shoulder_3: geometry collision mesh filename=file:///home/ubuntu/robot_ws/install/dual_arm_description/s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; visual mesh filename=file:///home/ubuntu/robot_ws/install/dual_arm_description/s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
- link shoulder_4: geometry collision mesh filename=file:///home/ubuntu/robot_ws/install/dual_arm_description/s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; visual mesh filename=file:///home/ubuntu/robot_ws/install/dual_arm_description/s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
- link shoulder_5: geometry collision mesh filename=file:///home/ubuntu/robot_ws/install/dual_arm_description/s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; visual mesh filename=file:///home/ubuntu/robot_ws/install/dual_arm_description/s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
- link shoulder_6: geometry collision mesh filename=file:///home/ubuntu/robot_ws/install/dual_arm_description/s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; visual mesh filename=file:///home/ubuntu/robot_ws/install/dual_arm_description/s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
- link wrist: geometry collision mesh filename=file:///home/ubuntu/robot_ws/install/dual_arm_description/s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; visual mesh filename=file:///home/ubuntu/robot_ws/install/dual_arm_description/s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
- link wristR: geometry collision mesh filename=file:///home/ubuntu/robot_ws/install/dual_arm_description/s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; visual mesh filename=file:///home/ubuntu/robot_ws/install/dual_arm_description/s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
Joints:
- added joint world_fixed: type fixed, parent world, child base_link, origin xyz=0 0 1.5 rpy=0 0 0
