Commit message: Update dual arm description and simulation

File: robotics/dual_arm_description/urdf/dual_arm.urdf.xacro (robot description, xacro)
@@ -3,6 +3,5 @@
      Commit Version: 1.6.0-4-g7f85cfe  Build Version: 1.6.7995.38578
      For more information, please see http://wiki.ros.org/sw_urdf_exporter -->
-<robot
-  name="dual_arm">
+<robot xmlns:xacro="http://www.ros.org/wiki/xacro" name="dual_arm">
   <link name="world"/>
   <joint name="world_fixed" type="fixed">
@@ -33,5 +32,5 @@
       <geometry>
         <mesh
-          filename="file:///home/ubuntu/robot_ws/install/dual_arm_description/share/dual_arm_description/meshes/base_link.STL" />
+          filename="file://$(find dual_arm_description)/meshes/base_link.STL" />
       </geometry>
       <material
@@ -47,5 +46,5 @@
       <geometry>
         <mesh
-          filename="file:///home/ubuntu/robot_ws/install/dual_arm_description/share/dual_arm_description/meshes/base_link.STL" />
+          filename="file://$(find dual_arm_description)/meshes/base_link.STL" />
       </geometry>
     </collision>
@@ -73,5 +72,5 @@
       <geometry>
         <mesh
-          filename="file:///home/ubuntu/robot_ws/install/dual_arm_description/share/dual_arm_description/meshes/pinion.STL" />
+          filename="file://$(find dual_arm_description)/meshes/pinion.STL" />
       </geometry>
       <material
@@ -87,5 +86,5 @@
       <geometry>
         <mesh
-          filename="file:///home/ubuntu/robot_ws/install/dual_arm_description/share/dual_arm_description/meshes/pinion.STL" />
+          filename="file://$(find dual_arm_description)/meshes/pinion.STL" />
       </geometry>
     </collision>
@@ -127,5 +126,5 @@
       <geometry>
         <mesh
-          filename="file:///home/ubuntu/robot_ws/install/dual_arm_description/share/dual_arm_description/meshes/rack.STL" />
+          filename="file://$(find dual_arm_description)/meshes/rack.STL" />
       </geometry>
       <material
@@ -141,5 +140,5 @@
       <geometry>
         <mesh
-          filename="file:///home/ubuntu/robot_ws/install/dual_arm_description/share/dual_arm_description/meshes/rack.STL" />
+          filename="file://$(find dual_arm_description)/meshes/rack.STL" />
       </geometry>
     </collision>
@@ -180,19 +179,19 @@
       <geometry>
         <mesh
-          filename="file:///home/ubuntu/robot_ws/install/dual_arm_description/share/dual_arm_description/meshes/robot_base.STL" />
-      </geometry>
-      <material
-        name="">
-        <color
-          rgba="0.650980392156863 0.619607843137255 0.588235294117647 1" />
-      </material>
-    </visual>
-    <collision>
-      <origin
-        xyz="0 0 0"
-        rpy="0 0 0" />
-      <geometry>
-        <mesh
-          filename="file:///home/ubuntu/robot_ws/install/dual_arm_description/share/dual_arm_description/meshes/robot_base.STL" />
+          filename="file://$(find dual_arm_description)/meshes/robot_base.STL" />
+      </geometry>
+      <material
+        name="">
+        <color
+          rgba="0.650980392156863 0.619607843137255 0.588235294117647 1" />
+      </material>
+    </visual>
+    <collision>
+      <origin
+        xyz="0 0 0"
+        rpy="0 0 0" />
+      <geometry>
+        <mesh
+          filename="file://$(find dual_arm_description)/meshes/robot_base.STL" />
       </geometry>
     </collision>
@@ -234,19 +233,19 @@
       <geometry>
         <mesh
-          filename="file:///home/ubuntu/robot_ws/install/dual_arm_description/share/dual_arm_description/meshes/shoulder_1.STL" />
-      </geometry>
-      <material
-        name="">
-        <color
-          rgba="0.650980392156863 0.619607843137255 0.588235294117647 1" />
-      </material>
-    </visual>
-    <collision>
-      <origin
-        xyz="0 0 0"
-        rpy="0 0 0" />
-      <geometry>
-        <mesh
-          filename="file:///home/ubuntu/robot_ws/install/dual_arm_description/share/dual_arm_description/meshes/shoulder_1.STL" />
+          filename="file://$(find dual_arm_description)/meshes/shoulder_1.STL" />
+      </geometry>
+      <material
+        name="">
+        <color
+          rgba="0.650980392156863 0.619607843137255 0.588235294117647 1" />
+      </material>
+    </visual>
+    <collision>
+      <origin
+        xyz="0 0 0"
+        rpy="0 0 0" />
+      <geometry>
+        <mesh
+          filename="file://$(find dual_arm_description)/meshes/shoulder_1.STL" />
       </geometry>
     </collision>
@@ -288,19 +287,19 @@
       <geometry>
         <mesh
-          filename="file:///home/ubuntu/robot_ws/install/dual_arm_description/share/dual_arm_description/meshes/shoulder_2.STL" />
-      </geometry>
-      <material
-        name="">
-        <color
-          rgba="0.650980392156863 0.619607843137255 0.588235294117647 1" />
-      </material>
-    </visual>
-    <collision>
-      <origin
-        xyz="0 0 0"
-        rpy="0 0 0" />
-      <geometry>
-        <mesh
-          filename="file:///home/ubuntu/robot_ws/install/dual_arm_description/share/dual_arm_description/meshes/shoulder_2.STL" />
+          filename="file://$(find dual_arm_description)/meshes/shoulder_2.STL" />
+      </geometry>
+      <material
+        name="">
+        <color
+          rgba="0.650980392156863 0.619607843137255 0.588235294117647 1" />
+      </material>
+    </visual>
+    <collision>
+      <origin
+        xyz="0 0 0"
+        rpy="0 0 0" />
+      <geometry>
+        <mesh
+          filename="file://$(find dual_arm_description)/meshes/shoulder_2.STL" />
       </geometry>
     </collision>
@@ -342,19 +341,19 @@
       <geometry>
         <mesh
-          filename="file:///home/ubuntu/robot_ws/install/dual_arm_description/share/dual_arm_description/meshes/shoulder_3.STL" />
-      </geometry>
-      <material
-        name="">
-        <color
-          rgba="0.650980392156863 0.619607843137255 0.588235294117647 1" />
-      </material>
-    </visual>
-    <collision>
-      <origin
-        xyz="0 0 0"
-        rpy="0 0 0" />
-      <geometry>
-        <mesh
-          filename="file:///home/ubuntu/robot_ws/install/dual_arm_description/share/dual_arm_description/meshes/shoulder_3.STL" />
+          filename="file://$(find dual_arm_description)/meshes/shoulder_3.STL" />
+      </geometry>
+      <material
+        name="">
+        <color
+          rgba="0.650980392156863 0.619607843137255 0.588235294117647 1" />
+      </material>
+    </visual>
+    <collision>
+      <origin
+        xyz="0 0 0"
+        rpy="0 0 0" />
+      <geometry>
+        <mesh
+          filename="file://$(find dual_arm_description)/meshes/shoulder_3.STL" />
       </geometry>
     </collision>
@@ -396,19 +395,19 @@
       <geometry>
         <mesh
-          filename="file:///home/ubuntu/robot_ws/install/dual_arm_description/share/dual_arm_description/meshes/shoulder_4.STL" />
-      </geometry>
-      <material
-        name="">
-        <color
-          rgba="0.650980392156863 0.619607843137255 0.588235294117647 1" />
-      </material>
-    </visual>
-    <collision>
-      <origin
-        xyz="0 0 0"
-        rpy="0 0 0" />
-      <geometry>
-        <mesh
-          filename="file:///home/ubuntu/robot_ws/install/dual_arm_description/share/dual_arm_description/meshes/shoulder_4.STL" />
+          filename="file://$(find dual_arm_description)/meshes/shoulder_4.STL" />
+      </geometry>
+      <material
+        name="">
+        <color
+          rgba="0.650980392156863 0.619607843137255 0.588235294117647 1" />
+      </material>
+    </visual>
+    <collision>
+      <origin
+        xyz="0 0 0"
+        rpy="0 0 0" />
+      <geometry>
+        <mesh
+          filename="file://$(find dual_arm_description)/meshes/shoulder_4.STL" />
       </geometry>
     </collision>
@@ -450,19 +449,19 @@
       <geometry>
         <mesh
-          filename="file:///home/ubuntu/robot_ws/install/dual_arm_description/share/dual_arm_description/meshes/shoulder_5.STL" />
-      </geometry>
-      <material
-        name="">
-        <color
-          rgba="0.650980392156863 0.619607843137255 0.588235294117647 1" />
-      </material>
-    </visual>
-    <collision>
-      <origin
-        xyz="0 0 0"
-        rpy="0 0 0" />
-      <geometry>
-        <mesh
-          filename="file:///home/ubuntu/robot_ws/install/dual_arm_description/share/dual_arm_description/meshes/shoulder_5.STL" />
+          filename="file://$(find dual_arm_description)/meshes/shoulder_5.STL" />
+      </geometry>
+      <material
+        name="">
+        <color
+          rgba="0.650980392156863 0.619607843137255 0.588235294117647 1" />
+      </material>
+    </visual>
+    <collision>
+      <origin
+        xyz="0 0 0"
+        rpy="0 0 0" />
+      <geometry>
+        <mesh
+          filename="file://$(find dual_arm_description)/meshes/shoulder_5.STL" />
       </geometry>
     </collision>
@@ -504,19 +503,19 @@
       <geometry>
         <mesh
-          filename="file:///home/ubuntu/robot_ws/install/dual_arm_description/share/dual_arm_description/meshes/shoulder_6.STL" />
-      </geometry>
-      <material
-        name="">
-        <color
-          rgba="0.650980392156863 0.619607843137255 0.588235294117647 1" />
-      </material>
-    </visual>
-    <collision>
-      <origin
-        xyz="0 0 0"
-        rpy="0 0 0" />
-      <geometry>
-        <mesh
-          filename="file:///home/ubuntu/robot_ws/install/dual_arm_description/share/dual_arm_description/meshes/shoulder_6.STL" />
+          filename="file://$(find dual_arm_description)/meshes/shoulder_6.STL" />
+      </geometry>
+      <material
+        name="">
+        <color
+          rgba="0.650980392156863 0.619607843137255 0.588235294117647 1" />
+      </material>
+    </visual>
+    <collision>
+      <origin
+        xyz="0 0 0"
+        rpy="0 0 0" />
+      <geometry>
+        <mesh
+          filename="file://$(find dual_arm_description)/meshes/shoulder_6.STL" />
       </geometry>
     </collision>
@@ -558,19 +557,19 @@
       <geometry>
         <mesh
-          filename="file:///home/ubuntu/robot_ws/install/dual_arm_description/share/dual_arm_description/meshes/wrist.STL" />
-      </geometry>
-      <material
-        name="">
-        <color
-          rgba="0.650980392156863 0.619607843137255 0.588235294117647 1" />
-      </material>
-    </visual>
-    <collision>
-      <origin
-        xyz="0 0 0"
-        rpy="0 0 0" />
-      <geometry>
-        <mesh
-          filename="file:///home/ubuntu/robot_ws/install/dual_arm_description/share/dual_arm_description/meshes/wrist.STL" />
+          filename="file://$(find dual_arm_description)/meshes/wrist.STL" />
+      </geometry>
+      <material
+        name="">
+        <color
+          rgba="0.650980392156863 0.619607843137255 0.588235294117647 1" />
+      </material>
+    </visual>
+    <collision>
+      <origin
+        xyz="0 0 0"
+        rpy="0 0 0" />
+      <geometry>
+        <mesh
+          filename="file://$(find dual_arm_description)/meshes/wrist.STL" />
       </geometry>
     </collision>
@@ -612,19 +611,19 @@
       <geometry>
         <mesh
-          filename="file:///home/ubuntu/robot_ws/install/dual_arm_description/share/dual_arm_description/meshes/shoulderR_1.STL" />
-      </geometry>
-      <material
-        name="">
-        <color
-          rgba="0.650980392156863 0.619607843137255 0.588235294117647 1" />
-      </material>
-    </visual>
-    <collision>
-      <origin
-        xyz="0 0 0"
-        rpy="0 0 0" />
-      <geometry>
-        <mesh
-          filename="file:///home/ubuntu/robot_ws/install/dual_arm_description/share/dual_arm_description/meshes/shoulderR_1.STL" />
+          filename="file://$(find dual_arm_description)/meshes/shoulderR_1.STL" />
+      </geometry>
+      <material
+        name="">
+        <color
+          rgba="0.650980392156863 0.619607843137255 0.588235294117647 1" />
+      </material>
+    </visual>
+    <collision>
+      <origin
+        xyz="0 0 0"
+        rpy="0 0 0" />
+      <geometry>
+        <mesh
+          filename="file://$(find dual_arm_description)/meshes/shoulderR_1.STL" />
       </geometry>
     </collision>
@@ -666,19 +665,19 @@
       <geometry>
         <mesh
-          filename="file:///home/ubuntu/robot_ws/install/dual_arm_description/share/dual_arm_description/meshes/shoulderR_2.STL" />
-      </geometry>
-      <material
-        name="">
-        <color
-          rgba="0.650980392156863 0.619607843137255 0.588235294117647 1" />
-      </material>
-    </visual>
-    <collision>
-      <origin
-        xyz="0 0 0"
-        rpy="0 0 0" />
-      <geometry>
-        <mesh
-          filename="file:///home/ubuntu/robot_ws/install/dual_arm_description/share/dual_arm_description/meshes/shoulderR_2.STL" />
+          filename="file://$(find dual_arm_description)/meshes/shoulderR_2.STL" />
+      </geometry>
+      <material
+        name="">
+        <color
+          rgba="0.650980392156863 0.619607843137255 0.588235294117647 1" />
+      </material>
+    </visual>
+    <collision>
+      <origin
+        xyz="0 0 0"
+        rpy="0 0 0" />
+      <geometry>
+        <mesh
+          filename="file://$(find dual_arm_description)/meshes/shoulderR_2.STL" />
       </geometry>
     </collision>
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
Commit message: Update dual arm URDF and raise effort limits to support arm weight

File: robotics/dual_arm_description/urdf/dual_arm.urdf.xacro (robot description, xacro)
@@ -263,5 +263,5 @@
     <axis
       xyz="0 1 0" />
-    <limit lower="-3.14159" upper="3.14159" effort="100" velocity="1.0"/>
+    <limit lower="-3.14159" upper="3.14159" effort="300" velocity="1.0"/>
   </joint>
   <link
@@ -317,5 +317,5 @@
     <axis
       xyz="0 0 1" />
-    <limit lower="-3.14159" upper="3.14159" effort="100" velocity="1.0"/>
+    <limit lower="-3.14159" upper="3.14159" effort="300" velocity="1.0"/>
   </joint>
   <link
@@ -371,5 +371,5 @@
     <axis
       xyz="0 1 0" />
-    <limit lower="-3.14159" upper="3.14159" effort="100" velocity="1.0"/>
+    <limit lower="-3.14159" upper="3.14159" effort="250" velocity="1.0"/>
   </joint>
   <link
@@ -425,5 +425,5 @@
     <axis
       xyz="0 0 1" />
-    <limit lower="-3.14159" upper="3.14159" effort="100" velocity="1.0"/>
+    <limit lower="-3.14159" upper="3.14159" effort="200" velocity="1.0"/>
   </joint>
   <link
@@ -479,5 +479,5 @@
     <axis
       xyz="0 1 0" />
-    <limit lower="-3.14159" upper="3.14159" effort="100" velocity="1.0"/>
+    <limit lower="-3.14159" upper="3.14159" effort="150" velocity="1.0"/>
   </joint>
   <link
@@ -533,5 +533,5 @@
     <axis
       xyz="0 0 1" />
-    <limit lower="-3.14159" upper="3.14159" effort="100" velocity="1.0"/>
+    <limit lower="-3.14159" upper="3.14159" effort="150" velocity="1.0"/>
   </joint>
   <link
@@ -641,5 +641,5 @@
     <axis
       xyz="0 1 0" />
-    <limit lower="-3.14159" upper="3.14159" effort="100" velocity="1.0"/>
+    <limit lower="-3.14159" upper="3.14159" effort="300" velocity="1.0"/>
   </joint>
   <link
@@ -695,5 +695,5 @@
     <axis
       xyz="0 0 1" />
-    <limit lower="-3.14159" upper="3.14159" effort="100" velocity="1.0"/>
+    <limit lower="-3.14159" upper="3.14159" effort="300" velocity="1.0"/>
   </joint>
   <link
@@ -749,5 +749,5 @@
     <axis
       xyz="0 1 0" />
-    <limit lower="-3.14159" upper="3.14159" effort="100" velocity="1.0"/>
+    <limit lower="-3.14159" upper="3.14159" effort="250" velocity="1.0"/>
   </joint>
   <link
@@ -803,5 +803,5 @@
     <axis
       xyz="0 0 1" />
-    <limit lower="-3.14159" upper="3.14159" effort="100" velocity="1.0"/>
+    <limit lower="-3.14159" upper="3.14159" effort="200" velocity="1.0"/>
   </joint>
   <link
@@ -857,5 +857,5 @@
     <axis
       xyz="0 1 0" />
-    <limit lower="-3.14159" upper="3.14159" effort="100" velocity="1.0"/>
+    <limit lower="-3.14159" upper="3.14159" effort="150" velocity="1.0"/>
   </joint>
   <link
@@ -911,5 +911,5 @@
     <axis
       xyz="0 0 1" />
-    <limit lower="-3.14159" upper="3.14159" effort="100" velocity="1.0"/>
+    <limit lower="-3.14159" upper="3.14159" effort="150" velocity="1.0"/>
   </joint>
   <link
@@ -971,71 +971,129 @@
       <plugin>gz_ros2_control/GazeboSimSystem</plugin>
     </hardware>
+    <!-- Left arm: heavy shoulder joints get stronger gains -->
     <joint name="shoulder1_joint">
-      <command_interface name="position"/>
+      <command_interface name="position">
+        <param name="p">200.0</param>
+        <param name="i">0.0</param>
+        <param name="d">20.0</param>
+      </command_interface>
       <state_interface name="position"/>
       <state_interface name="velocity"/>
     </joint>
     <joint name="shoulder2_joint">
-      <command_interface name="position"/>
+      <command_interface name="position">
+        <param name="p">200.0</param>
+        <param name="i">0.0</param>
+        <param name="d">20.0</param>
+      </command_interface>
       <state_interface name="position"/>
       <state_interface name="velocity"/>
     </joint>
     <joint name="shoulder3_joint">
-      <command_interface name="position"/>
+      <command_interface name="position">
+        <param name="p">200.0</param>
+        <param name="i">0.0</param>
+        <param name="d">20.0</param>
+      </command_interface>
       <state_interface name="position"/>
       <state_interface name="velocity"/>
     </joint>
     <joint name="shoulder4_joint">
-      <command_interface name="position"/>
+      <command_interface name="position">
+        <param name="p">100.0</param>
+        <param name="i">0.0</param>
+        <param name="d">10.0</param>
+      </command_interface>
       <state_interface name="position"/>
       <state_interface name="velocity"/>
     </joint>
     <joint name="shoulder5_joint">
-      <command_interface name="position"/>
+      <command_interface name="position">
+        <param name="p">100.0</param>
+        <param name="i">0.0</param>
+        <param name="d">10.0</param>
+      </command_interface>
       <state_interface name="position"/>
       <state_interface name="velocity"/>
     </joint>
     <joint name="shoulder6_joint">
-      <command_interface name="position"/>
+      <command_interface name="position">
+        <param name="p">100.0</param>
+        <param name="i">0.0</param>
+        <param name="d">10.0</param>
+      </command_interface>
       <state_interface name="position"/>
       <state_interface name="velocity"/>
     </joint>
     <joint name="wrist_joint">
-      <command_interface name="position"/>
-      <state_interface name="position"/>
-      <state_interface name="velocity"/>
-    </joint>
+      <command_interface name="position">
+        <param name="p">80.0</param>
+        <param name="i">0.0</param>
+        <param name="d">8.0</param>
+      </command_interface>
+      <state_interface name="position"/>
+      <state_interface name="velocity"/>
+    </joint>
+    <!-- Right arm: same tiered gains, mirrored -->
     <joint name="shoulderR_joint">
-      <command_interface name="position"/>
+      <command_interface name="position">
+        <param name="p">200.0</param>
+        <param name="i">0.0</param>
+        <param name="d">20.0</param>
+      </command_interface>
       <state_interface name="position"/>
       <state_interface name="velocity"/>
     </joint>
     <joint name="shoulderR_2_joint">
-      <command_interface name="position"/>
+      <command_interface name="position">
+        <param name="p">200.0</param>
+        <param name="i">0.0</param>
+        <param name="d">20.0</param>
+      </command_interface>
       <state_interface name="position"/>
       <state_interface name="velocity"/>
     </joint>
     <joint name="shoulderR_3joint">
-      <command_interface name="position"/>
+      <command_interface name="position">
+        <param name="p">200.0</param>
+        <param name="i">0.0</param>
+        <param name="d">20.0</param>
+      </command_interface>
       <state_interface name="position"/>
       <state_interface name="velocity"/>
     </joint>
     <joint name="shoulderR_4joint">
-      <command_interface name="position"/>
+      <command_interface name="position">
+        <param name="p">100.0</param>
+        <param name="i">0.0</param>
+        <param name="d">10.0</param>
+      </command_interface>
       <state_interface name="position"/>
       <state_interface name="velocity"/>
     </joint>
     <joint name="shoulderR_5joint">
-      <command_interface name="position"/>
+      <command_interface name="position">
+        <param name="p">100.0</param>
+        <param name="i">0.0</param>
+        <param name="d">10.0</param>
+      </command_interface>
       <state_interface name="position"/>
       <state_interface name="velocity"/>
     </joint>
     <joint name="shoulderR_6joint">
-      <command_interface name="position"/>
+      <command_interface name="position">
+        <param name="p">100.0</param>
+        <param name="i">0.0</param>
+        <param name="d">10.0</param>
+      </command_interface>
       <state_interface name="position"/>
       <state_interface name="velocity"/>
     </joint>
     <joint name="wristR_joint">
-      <command_interface name="position"/>
+      <command_interface name="position">
+        <param name="p">80.0</param>
+        <param name="i">0.0</param>
+        <param name="d">8.0</param>
+      </command_interface>
       <state_interface name="position"/>
       <state_interface name="velocity"/>
