Commit message: corrected the URDF implementation of the pinion rack mechanical system and tested it in gazebo and it is working.

File: robotics/dual_arm_description/urdf/dual_arm.urdf.xacro (robot description, xacro)
@@ -4,5 +4,4 @@
      For more information, please see http://wiki.ros.org/sw_urdf_exporter -->
 <robot xmlns:xacro="http://www.ros.org/wiki/xacro" name="dual_arm">
-  <xacro:arg name="controllers_file" default=""/>
   <link name="world"/>
   <joint name="world_fixed" type="fixed">
@@ -33,5 +32,5 @@
       <geometry>
         <mesh
-          filename="package://dual_arm_description/meshes/base_link.STL" />
+          filename="file://$(find dual_arm_description)/meshes/base_link.STL" />
       </geometry>
       <material
@@ -47,5 +46,5 @@
       <geometry>
         <mesh
-          filename="package://dual_arm_description/meshes/base_link.STL" />
+          filename="file://$(find dual_arm_description)/meshes/base_link.STL" />
       </geometry>
     </collision>
@@ -73,5 +72,5 @@
       <geometry>
         <mesh
-          filename="package://dual_arm_description/meshes/pinion.STL" />
+          filename="file://$(find dual_arm_description)/meshes/pinion.STL" />
       </geometry>
       <material
@@ -87,5 +86,5 @@
       <geometry>
         <mesh
-          filename="package://dual_arm_description/meshes/pinion.STL" />
+          filename="file://$(find dual_arm_description)/meshes/pinion.STL" />
       </geometry>
     </collision>
@@ -103,5 +102,5 @@
     <axis
       xyz="1 0 0" />
-    <limit lower="-3.14159" upper="3.14159" effort="100" velocity="1.0"/>
+    <limit lower="0.0" upper="7.2" effort="1000" velocity="20.0"/>
   </joint>
   <link
@@ -127,5 +126,5 @@
       <geometry>
         <mesh
-          filename="package://dual_arm_description/meshes/rack.STL" />
+          filename="file://$(find dual_arm_description)/meshes/rack.STL" />
       </geometry>
       <material
@@ -141,5 +140,5 @@
       <geometry>
         <mesh
-          filename="package://dual_arm_description/meshes/rack.STL" />
+          filename="file://$(find dual_arm_description)/meshes/rack.STL" />
       </geometry>
     </collision>
@@ -155,6 +154,7 @@
         lower="-0.40"
         upper="0"
-        effort="100"
-        velocity="1.0"/>
+        effort="15000"
+        velocity="5.0"/>
+    <mimic joint="pinion_joint" multiplier="-0.056" offset="0.0"/>
 </joint>
   <link
@@ -180,19 +180,19 @@
       <geometry>
         <mesh
-          filename="package://dual_arm_description/meshes/robot_base.STL" />
-      </geometry>
-      <material
-        name="">
-        <color
-          rgba="0.650980392156863 0.619607843137255 0.588235294117647 1" />
-      </material>
-    </visual>
-    <collision>
-      <origin
-        xyz="0 0 0"
-        rpy="0 0 0" />
-      <geometry>
-        <mesh
-          filename="package://dual_arm_description/meshes/robot_base.STL" />
+          filename="file://$(find dual_arm_description)/meshes/robot_base.STL" />
+      </geometry>
+      <material
+        name="">
+        <color
+          rgba="0.650980392156863 0.619607843137255 0.588235294117647 1" />
+      </material>
+    </visual>
+    <collision>
+      <origin
+        xyz="0 0 0"
+        rpy="0 0 0" />
+      <geometry>
+        <mesh
+          filename="file://$(find dual_arm_description)/meshes/robot_base.STL" />
       </geometry>
     </collision>
@@ -210,5 +210,5 @@
     <axis
       xyz="0 0 1" />
-    <limit lower="-3.14159" upper="3.14159" effort="100" velocity="1.0"/>
+    <limit lower="-3.14159" upper="3.14159" effort="500" velocity="1.0"/>
   </joint>
   <link
@@ -234,19 +234,19 @@
       <geometry>
         <mesh
-          filename="package://dual_arm_description/meshes/shoulder_1.STL" />
-      </geometry>
-      <material
-        name="">
-        <color
-          rgba="0.650980392156863 0.619607843137255 0.588235294117647 1" />
-      </material>
-    </visual>
-    <collision>
-      <origin
-        xyz="0 0 0"
-        rpy="0 0 0" />
-      <geometry>
-        <mesh
-          filename="package://dual_arm_description/meshes/shoulder_1.STL" />
+          filename="file://$(find dual_arm_description)/meshes/shoulder_1.STL" />
+      </geometry>
+      <material
+        name="">
+        <color
+          rgba="0.650980392156863 0.619607843137255 0.588235294117647 1" />
+      </material>
+    </visual>
+    <collision>
+      <origin
+        xyz="0 0 0"
+        rpy="0 0 0" />
+      <geometry>
+        <mesh
+          filename="file://$(find dual_arm_description)/meshes/shoulder_1.STL" />
       </geometry>
     </collision>
@@ -288,19 +288,19 @@
       <geometry>
         <mesh
-          filename="package://dual_arm_description/meshes/shoulder_2.STL" />
-      </geometry>
-      <material
-        name="">
-        <color
-          rgba="0.650980392156863 0.619607843137255 0.588235294117647 1" />
-      </material>
-    </visual>
-    <collision>
-      <origin
-        xyz="0 0 0"
-        rpy="0 0 0" />
-      <geometry>
-        <mesh
-          filename="package://dual_arm_description/meshes/shoulder_2.STL" />
+          filename="file://$(find dual_arm_description)/meshes/shoulder_2.STL" />
+      </geometry>
+      <material
+        name="">
+        <color
+          rgba="0.650980392156863 0.619607843137255 0.588235294117647 1" />
+      </material>
+    </visual>
+    <collision>
+      <origin
+        xyz="0 0 0"
+        rpy="0 0 0" />
+      <geometry>
+        <mesh
+          filename="file://$(find dual_arm_description)/meshes/shoulder_2.STL" />
       </geometry>
     </collision>
@@ -342,19 +342,19 @@
       <geometry>
         <mesh
-          filename="package://dual_arm_description/meshes/shoulder_3.STL" />
-      </geometry>
-      <material
-        name="">
-        <color
-          rgba="0.650980392156863 0.619607843137255 0.588235294117647 1" />
-      </material>
-    </visual>
-    <collision>
-      <origin
-        xyz="0 0 0"
-        rpy="0 0 0" />
-      <geometry>
-        <mesh
-          filename="package://dual_arm_description/meshes/shoulder_3.STL" />
+          filename="file://$(find dual_arm_description)/meshes/shoulder_3.STL" />
+      </geometry>
+      <material
+        name="">
+        <color
+          rgba="0.650980392156863 0.619607843137255 0.588235294117647 1" />
+      </material>
+    </visual>
+    <collision>
+      <origin
+        xyz="0 0 0"
+        rpy="0 0 0" />
+      <geometry>
+        <mesh
+          filename="file://$(find dual_arm_description)/meshes/shoulder_3.STL" />
       </geometry>
     </collision>
@@ -396,19 +396,19 @@
       <geometry>
         <mesh
-          filename="package://dual_arm_description/meshes/shoulder_4.STL" />
-      </geometry>
-      <material
-        name="">
-        <color
-          rgba="0.650980392156863 0.619607843137255 0.588235294117647 1" />
-      </material>
-    </visual>
-    <collision>
-      <origin
-        xyz="0 0 0"
-        rpy="0 0 0" />
-      <geometry>
-        <mesh
-          filename="package://dual_arm_description/meshes/shoulder_4.STL" />
+          filename="file://$(find dual_arm_description)/meshes/shoulder_4.STL" />
+      </geometry>
+      <material
+        name="">
+        <color
+          rgba="0.650980392156863 0.619607843137255 0.588235294117647 1" />
+      </material>
+    </visual>
+    <collision>
+      <origin
+        xyz="0 0 0"
+        rpy="0 0 0" />
+      <geometry>
+        <mesh
+          filename="file://$(find dual_arm_description)/meshes/shoulder_4.STL" />
       </geometry>
     </collision>
@@ -450,19 +450,19 @@
       <geometry>
         <mesh
-          filename="package://dual_arm_description/meshes/shoulder_5.STL" />
-      </geometry>
-      <material
-        name="">
-        <color
-          rgba="0.650980392156863 0.619607843137255 0.588235294117647 1" />
-      </material>
-    </visual>
-    <collision>
-      <origin
-        xyz="0 0 0"
-        rpy="0 0 0" />
-      <geometry>
-        <mesh
-          filename="package://dual_arm_description/meshes/shoulder_5.STL" />
+          filename="file://$(find dual_arm_description)/meshes/shoulder_5.STL" />
+      </geometry>
+      <material
+        name="">
+        <color
+          rgba="0.650980392156863 0.619607843137255 0.588235294117647 1" />
+      </material>
+    </visual>
+    <collision>
+      <origin
+        xyz="0 0 0"
+        rpy="0 0 0" />
+      <geometry>
+        <mesh
+          filename="file://$(find dual_arm_description)/meshes/shoulder_5.STL" />
       </geometry>
     </collision>
@@ -504,19 +504,19 @@
       <geometry>
         <mesh
-          filename="package://dual_arm_description/meshes/shoulder_6.STL" />
-      </geometry>
-      <material
-        name="">
-        <color
-          rgba="0.650980392156863 0.619607843137255 0.588235294117647 1" />
-      </material>
-    </visual>
-    <collision>
-      <origin
-        xyz="0 0 0"
-        rpy="0 0 0" />
-      <geometry>
-        <mesh
-          filename="package://dual_arm_description/meshes/shoulder_6.STL" />
+          filename="file://$(find dual_arm_description)/meshes/shoulder_6.STL" />
+      </geometry>
+      <material
+        name="">
+        <color
+          rgba="0.650980392156863 0.619607843137255 0.588235294117647 1" />
+      </material>
+    </visual>
+    <collision>
+      <origin
+        xyz="0 0 0"
+        rpy="0 0 0" />
+      <geometry>
+        <mesh
+          filename="file://$(find dual_arm_description)/meshes/shoulder_6.STL" />
       </geometry>
     </collision>
@@ -558,19 +558,19 @@
       <geometry>
         <mesh
-          filename="package://dual_arm_description/meshes/wrist.STL" />
-      </geometry>
-      <material
-        name="">
-        <color
-          rgba="0.650980392156863 0.619607843137255 0.588235294117647 1" />
-      </material>
-    </visual>
-    <collision>
-      <origin
-        xyz="0 0 0"
-        rpy="0 0 0" />
-      <geometry>
-        <mesh
-          filename="package://dual_arm_description/meshes/wrist.STL" />
+          filename="file://$(find dual_arm_description)/meshes/wrist.STL" />
+      </geometry>
+      <material
+        name="">
+        <color
+          rgba="0.650980392156863 0.619607843137255 0.588235294117647 1" />
+      </material>
+    </visual>
+    <collision>
+      <origin
+        xyz="0 0 0"
+        rpy="0 0 0" />
+      <geometry>
+        <mesh
+          filename="file://$(find dual_arm_description)/meshes/wrist.STL" />
       </geometry>
     </collision>
@@ -612,19 +612,19 @@
       <geometry>
         <mesh
-          filename="package://dual_arm_description/meshes/shoulderR_1.STL" />
-      </geometry>
-      <material
-        name="">
-        <color
-          rgba="0.650980392156863 0.619607843137255 0.588235294117647 1" />
-      </material>
-    </visual>
-    <collision>
-      <origin
-        xyz="0 0 0"
-        rpy="0 0 0" />
-      <geometry>
-        <mesh
-          filename="package://dual_arm_description/meshes/shoulderR_1.STL" />
+          filename="file://$(find dual_arm_description)/meshes/shoulderR_1.STL" />
+      </geometry>
+      <material
+        name="">
+        <color
+          rgba="0.650980392156863 0.619607843137255 0.588235294117647 1" />
+      </material>
+    </visual>
+    <collision>
+      <origin
+        xyz="0 0 0"
+        rpy="0 0 0" />
+      <geometry>
+        <mesh
+          filename="file://$(find dual_arm_description)/meshes/shoulderR_1.STL" />
       </geometry>
     </collision>
@@ -666,19 +666,19 @@
       <geometry>
         <mesh
-          filename="package://dual_arm_description/meshes/shoulderR_2.STL" />
-      </geometry>
-      <material
-        name="">
-        <color
-          rgba="0.650980392156863 0.619607843137255 0.588235294117647 1" />
-      </material>
-    </visual>
-    <collision>
-      <origin
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
Commit message: Fix rack-pinion mimic coupling (Bullet-Featherstone), add robot_base_joint controller

File: robotics/dual_arm_description/urdf/dual_arm.urdf.xacro (robot description, xacro)
@@ -102,5 +102,5 @@
     <axis
       xyz="1 0 0" />
-    <limit lower="-3.14159" upper="3.14159" effort="100" velocity="1.0"/>
+    <limit lower="0.0" upper="7.2" effort="1000" velocity="20.0"/>
   </joint>
   <link
@@ -154,6 +154,7 @@
         lower="-0.40"
         upper="0"
-        effort="100"
-        velocity="1.0"/>
+        effort="15000"
+        velocity="5.0"/>
+    <mimic joint="pinion_joint" multiplier="-0.056" offset="0.0"/>
 </joint>
   <link
@@ -209,5 +210,5 @@
     <axis
       xyz="0 0 1" />
-    <limit lower="-3.14159" upper="3.14159" effort="100" velocity="1.0"/>
+    <limit lower="-3.14159" upper="3.14159" effort="500" velocity="1.0"/>
   </joint>
   <link
@@ -971,4 +972,28 @@
       <plugin>gz_ros2_control/GazeboSimSystem</plugin>
     </hardware>
+    <joint name="pinion_joint">
+      <command_interface name="position">
+        <param name="p">1500.0</param>
+        <param name="i">200.0</param>
+        <param name="d">10.0</param>
+      </command_interface>
+      <state_interface name="position"/>
+      <state_interface name="velocity"/>
+    </joint>
+    <joint name="rack_joint">
+      <param name="mimic">pinion_joint</param>
+      <param name="multiplier">-0.056</param>
+      <state_interface name="position"/>
+      <state_interface name="velocity"/>
+    </joint>
+    <joint name="robot_base_joint">
+      <command_interface name="position">
+        <param name="p">300.0</param>
+        <param name="i">0.0</param>
+        <param name="d">30.0</param>
+      </command_interface>
+      <state_interface name="position"/>
+      <state_interface name="velocity"/>
+    </joint>
     <!-- Left arm: heavy shoulder joints get stronger gains -->
     <joint name="shoulder1_joint">

Commit message: Fix moveit configuration to enable lift and base groups planning and execution

File: robotics/dual_arm_description/urdf/dual_arm.urdf.xacro (robot description, xacro)
@@ -102,5 +102,5 @@
     <axis
       xyz="1 0 0" />
-    <limit lower="0.0" upper="7.2" effort="1000" velocity="20.0"/>
+    <limit lower="-0.001" upper="7.2" effort="1000" velocity="20.0"/>
   </joint>
   <link

Commit message: Fix arms instability by matching effort limits in moveit with urdf

File: robotics/dual_arm_description/urdf/dual_arm.urdf.xacro (robot description, xacro)
@@ -985,5 +985,5 @@
       <command_interface name="position">
         <param name="p">300.0</param>
-        <param name="i">0.0</param>
+        <param name="i">10.0</param>
         <param name="d">30.0</param>
       </command_interface>
@@ -991,10 +991,9 @@
       <state_interface name="velocity"/>
     </joint>
-    <!-- Left arm: heavy shoulder joints get stronger gains -->
     <joint name="shoulder1_joint">
       <command_interface name="position">
-        <param name="p">200.0</param>
-        <param name="i">0.0</param>
-        <param name="d">20.0</param>
+        <param name="p">350.0</param>
+        <param name="i">30.0</param>
+        <param name="d">35.0</param>
       </command_interface>
       <state_interface name="position"/>
@@ -1003,7 +1002,7 @@
     <joint name="shoulder2_joint">
       <command_interface name="position">
-        <param name="p">200.0</param>
-        <param name="i">0.0</param>
-        <param name="d">20.0</param>
+        <param name="p">350.0</param>
+        <param name="i">30.0</param>
+        <param name="d">35.0</param>
       </command_interface>
       <state_interface name="position"/>
@@ -1012,7 +1011,7 @@
     <joint name="shoulder3_joint">
       <command_interface name="position">
-        <param name="p">200.0</param>
-        <param name="i">0.0</param>
-        <param name="d">20.0</param>
+        <param name="p">280.0</param>
+        <param name="i">20.0</param>
+        <param name="d">28.0</param>
       </command_interface>
       <state_interface name="position"/>
@@ -1021,7 +1020,7 @@
     <joint name="shoulder4_joint">
       <command_interface name="position">
-        <param name="p">100.0</param>
-        <param name="i">0.0</param>
-        <param name="d">10.0</param>
+        <param name="p">160.0</param>
+        <param name="i">12.0</param>
+        <param name="d">16.0</param>
       </command_interface>
       <state_interface name="position"/>
@@ -1030,7 +1029,7 @@
     <joint name="shoulder5_joint">
       <command_interface name="position">
-        <param name="p">100.0</param>
-        <param name="i">0.0</param>
-        <param name="d">10.0</param>
+        <param name="p">160.0</param>
+        <param name="i">12.0</param>
+        <param name="d">16.0</param>
       </command_interface>
       <state_interface name="position"/>
@@ -1039,7 +1038,7 @@
     <joint name="shoulder6_joint">
       <command_interface name="position">
-        <param name="p">100.0</param>
-        <param name="i">0.0</param>
-        <param name="d">10.0</param>
+        <param name="p">140.0</param>
+        <param name="i">8.0</param>
+        <param name="d">14.0</param>
       </command_interface>
       <state_interface name="position"/>
@@ -1048,17 +1047,17 @@
     <joint name="wrist_joint">
       <command_interface name="position">
-        <param name="p">80.0</param>
-        <param name="i">0.0</param>
-        <param name="d">8.0</param>
-      </command_interface>
-      <state_interface name="position"/>
-      <state_interface name="velocity"/>
-    </joint>
-    <!-- Right arm: same tiered gains, mirrored -->
+        <param name="p">120.0</param>
+        <param name="i">6.0</param>
+        <param name="d">12.0</param>
+      </command_interface>
+      <state_interface name="position"/>
+      <state_interface name="velocity"/>
+    </joint>
+    <!-- Right arm: same boosted, mirrored gains -->
     <joint name="shoulderR_joint">
       <command_interface name="position">
-        <param name="p">200.0</param>
-        <param name="i">0.0</param>
-        <param name="d">20.0</param>
+        <param name="p">350.0</param>
+        <param name="i">30.0</param>
+        <param name="d">35.0</param>
       </command_interface>
       <state_interface name="position"/>
@@ -1067,7 +1066,7 @@
     <joint name="shoulderR_2_joint">
       <command_interface name="position">
-        <param name="p">200.0</param>
-        <param name="i">0.0</param>
-        <param name="d">20.0</param>
+        <param name="p">350.0</param>
+        <param name="i">30.0</param>
+        <param name="d">35.0</param>
       </command_interface>
       <state_interface name="position"/>
@@ -1076,7 +1075,7 @@
     <joint name="shoulderR_3joint">
       <command_interface name="position">
-        <param name="p">200.0</param>
-        <param name="i">0.0</param>
-        <param name="d">20.0</param>
+        <param name="p">280.0</param>
+        <param name="i">20.0</param>
+        <param name="d">28.0</param>
       </command_interface>
       <state_interface name="position"/>
@@ -1085,7 +1084,7 @@
     <joint name="shoulderR_4joint">
       <command_interface name="position">
-        <param name="p">100.0</param>
-        <param name="i">0.0</param>
-        <param name="d">10.0</param>
+        <param name="p">160.0</param>
+        <param name="i">12.0</param>
+        <param name="d">16.0</param>
       </command_interface>
       <state_interface name="position"/>
@@ -1094,7 +1093,7 @@
     <joint name="shoulderR_5joint">
       <command_interface name="position">
-        <param name="p">100.0</param>
-        <param name="i">0.0</param>
-        <param name="d">10.0</param>
+        <param name="p">160.0</param>
+        <param name="i">12.0</param>
+        <param name="d">16.0</param>
       </command_interface>
       <state_interface name="position"/>
@@ -1103,7 +1102,7 @@
     <joint name="shoulderR_6joint">
       <command_interface name="position">
-        <param name="p">100.0</param>
-        <param name="i">0.0</param>
-        <param name="d">10.0</param>
+        <param name="p">140.0</param>
+        <param name="i">8.0</param>
+        <param name="d">14.0</param>
       </command_interface>
       <state_interface name="position"/>
@@ -1112,7 +1111,7 @@
     <joint name="wristR_joint">
       <command_interface name="position">
-        <param name="p">80.0</param>
-        <param name="i">0.0</param>
-        <param name="d">8.0</param>
+        <param name="p">120.0</param>
+        <param name="i">6.0</param>
+        <param name="d">12.0</param>
       </command_interface>
       <state_interface name="position"/>
